Commit message: feat:实现了nav goal进行导航

File: mas2027_robot_description/urdf/mas2027_sentry.urdf (robot description, URDF)
Before this commit: robot mas2027_sentry, 5 links, 4 joints
Links:
- removed link lakibeam_frame
Joints:
- removed joint lakibeam_joint
- joint lidar_joint: origin xyz=0.09 0.03 0.11 rpy=0.3572 0 1.5708 -> xyz=0.09 0.03 0.11 rpy=0.5046 0 1.5708

Commit message: feat:修正雷达外参，加入离线建图

File: mas2027_robot_description/urdf/mas2027_sentry.urdf (robot description, URDF)
Before this commit: robot mas2027_sentry, 4 links, 3 joints
Joints:
- joint lidar_joint: origin xyz=0.09 0.03 0.11 rpy=0.5046 0 1.5708 -> xyz=0.09 0.03 0.11 rpy=0.8389 0 1.5708

Commit message: feat:加入了有先验点云下的重定位修改了车体模型

File: mas2027_robot_description/urdf/mas2027_sentry.urdf (robot description, URDF)
Before this commit: robot mas2027_sentry, 4 links, 3 joints
Joints:
- joint lidar_joint: origin xyz=0.09 0.03 0.11 rpy=0.8389 0 1.5708 -> xyz=0.00 -0.15 0.11 rpy=0.8389 0 0

Commit message: feat：修改

File: mas2027_robot_description/urdf/mas2027_sentry.urdf (robot description, URDF)
Before this commit: robot mas2027_sentry, 4 links, 3 joints
Links:
- added link lidar_back_link; visual mesh filename=package://mas2027_robot_description/meshes/mid360.STL
Joints:
- added joint lidar_back_joint: type fixed, parent base_link, child lidar_back_link, origin xyz=0.00 0.15 0.11 rpy=-0.8389 0 0
